File: NES-IO/PCB_EU/NES_IO_EU.brd (EAGLE design)
At the start: 72.8 x 77.5 mm, 66 parts, among them IC1 74HC125D, J1.1 MY_JUMPER, J1.2 MY_JUMPER, J2.2 10k, J4.C MY_JUMPER, J4.V MY_JUMPER, J6 MY_JUMPER, J7 MY_JUMPER

Commit message: Update PCB and its name (EU version)
Routing:
- net N$31: track 29.9 -> 33.6 mm
- net N$16: vias 1 -> 0
- net N$15: vias 1 -> 0
Other:
- board text added: ")"
- board text added: "/"
- board text added: "4"
- board text added: "8"
- board text added: "9"
- board text added: "Version: 20151228EU"
- board text added: "_"
- board text added: "b"
- board text added: "i"
- board text added: "o"
- board text added: "r"
- board text added: "t"
- board text removed: "Version: 20151220EU"
Changed lines of the file:
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@@
 <wire x1="59.055" y1="43.02125" x2="12.7" y2="43.02125" width="0.1524" layer="26"/>
 <text x="71.755" y="67.15125" size="1.27" layer="26" font="vector" ratio="12" rot="MR0">Version:
-20151220EU</text>
+20151228EU</text>
 <wire x1="71.755" y1="68.73875" x2="63.8175" y2="68.73875" width="0.1524" layer="26" style="shortdash"/>
 <wire x1="59.055" y1="5.715" x2="59.055" y2="0.635" width="0.1524" layer="25" style="shortdash"/>
@@
 <wire x1="67.945" y1="32.54375" x2="67.6275" y2="32.86125" width="0.1524" layer="21"/>
 <wire x1="69.05625" y1="35.2425" x2="66.19875" y2="35.2425" width="0.1524" layer="21"/>
+<text x="32.987840625" y="34.9630125" size="1.524" layer="29" font="vector" ratio="20">b</text>
+<text x="34.284140625" y="34.955475" size="1.524" layer="29" font="vector" ratio="20">o</text>
+<text x="35.60305" y="34.9479375" size="1.524" layer="29" font="vector" ratio="20">r</text>
+<text x="36.688325" y="34.940403125" size="1.524" layer="29" font="vector" ratio="20">t</text>
+<text x="37.5550375" y="34.9479375" size="1.524" layer="29" font="vector" ratio="20">i</text>
+<text x="38.4292875" y="34.9479375" size="1.524" layer="29" font="vector" ratio="20">4</text>
+<text x="39.733125" y="34.9479375" size="1.524" layer="29" font="vector" ratio="20">9</text>
+<text x="41.052034375" y="34.9479375" size="1.524" layer="29" font="vector" ratio="20">3</text>
+<text x="42.363409375" y="34.9479375" size="1.524" layer="29" font="vector" ratio="20">8</text>
+<text x="32.965228125" y="32.8150375" size="1.524" layer="29" font="vector" ratio="20">_</text>
+<text x="34.284140625" y="32.8150375" size="1.524" layer="29" font="vector" ratio="20">_</text>
+<text x="37.7736" y="32.8150375" size="1.524" layer="29" font="vector" ratio="20">_</text>
+<text x="39.0925125" y="32.8150375" size="1.524" layer="29" font="vector" ratio="20">_</text>
+<text x="42.581971875" y="32.8150375" size="1.524" layer="29" font="vector" ratio="20">_</text>
+<text x="40.3888125" y="32.8150375" size="1.524" layer="29" font="vector" ratio="20">/</text>
+<text x="35.580440625" y="32.8150375" size="1.524" layer="29" font="vector" ratio="20">/</text>
+<text x="36.89935" y="32.8150375" size="1.524" layer="29" font="vector" ratio="20">)</text>
+<text x="41.69265" y="32.822575" size="1.524" layer="29" font="vector" ratio="20">)</text>
 </plain>
 <attributes>
@@
 <via x="60.48375" y="14.605" extent="1-16" drill="0.6"/>
 <via x="62.865" y="9.2075" extent="1-16" drill="0.6"/>
-<via x="30.48" y="40.64" extent="1-16" drill="0.6"/>
+<via x="26.67" y="38.735" extent="1-16" drill="0.6"/>
 <via x="46.355" y="36.195" extent="1-16" drill="0.6"/>
 <via x="42.545" y="49.53" extent="1-16" drill="0.6"/>
@@
 <signal name="N$15">
 <contactref element="R1" pad="1"/>
-<via x="60.325" y="3.33375" extent="1-16" drill="1"/>
 <contactref element="U$14" pad="P$1"/>
 <contactref element="U$14" pad="P$2"/>
@@
 <signal name="N$16">
 <contactref element="R2" pad="1"/>
-<via x="65.405" y="3.33375" extent="1-16" drill="1"/>
 <contactref element="U$15" pad="P$1"/>
 <contactref element="U$15" pad="P$2"/>
@@
 <contactref element="J7" pad="P$1"/>
 <wire x1="33.34" y1="41.91" x2="30.3784" y2="41.91" width="0.4064" layer="1"/>
-<wire x1="33.34" y1="41.91" x2="33.34" y2="43.01875" width="0.4064" layer="1"/>
-<wire x1="33.34" y1="43.01875" x2="32.54375" y2="43.815" width="0.4064" layer="1"/>
-<via x="32.54375" y="43.815" extent="1-16" drill="0.6"/>
+<wire x1="33.34" y1="41.91" x2="33.34" y2="40.955" width="0.4064" layer="1"/>
+<wire x1="33.34" y1="40.955" x2="32.385" y2="40.005" width="0.4064" layer="1"/>
+<via x="32.385" y="40.005" extent="1-16" drill="0.6"/>
 <wire x1="30.48" y1="52.07" x2="31.75" y2="53.34" width="0.4064" layer="1"/>
 <wire x1="31.75" y1="53.34" x2="38.735" y2="53.34" width="0.4064" layer="1"/>
@@
 <wire x1="39.6875" y1="52.3875" x2="39.6875" y2="49.53" width="0.4064" layer="1"/>
 <wire x1="30.48" y1="52.07" x2="29.21" y2="50.8" width="0.4064" layer="16"/>
-<wire x1="29.21" y1="50.8" x2="29.21" y2="44.45" width="0.4064" layer="16"/>
-<wire x1="29.21" y1="44.45" x2="29.845" y2="43.815" width="0.4064" layer="16"/>
-<wire x1="29.845" y1="43.815" x2="32.54375" y2="43.815" width="0.4064" layer="16"/>
+<wire x1="29.21" y1="50.8" x2="29.21" y2="40.64" width="0.4064" layer="16"/>
+<wire x1="29.21" y1="40.64" x2="29.845" y2="40.005" width="0.4064" layer="16"/>
+<wire x1="29.845" y1="40.005" x2="32.385" y2="40.005" width="0.4064" layer="16"/>
 </signal>
 <signal name="N$32">

Commit message: Update PCB files
Routing:
- net GND: track 36.5 -> 130.0 mm, vias 92 -> 90
- net AC2: track 26.9 -> 46.1 mm
- net AC1B: track 14.2 -> 33.4 mm
- net VCC: track 155.1 -> 166.8 mm
- net AC1A: track 18.5 -> 30.1 mm
- net DC2: track 142.7 -> 147.6 mm
- net DC1: track 52.7 -> 55.9 mm
- net N$5: track 126.9 -> 125.4 mm
- net N$29: track 69.5 -> 68.2 mm
- net N$32: track 21.5 -> 22.6 mm
- net N$12: track 68.1 -> 68.8 mm
Other:
- board text added: "Version: 20160420EU"
- board text removed: "Version: 20151228EU"
