File: NES-IO/PCB_US/NES_IO_US.brd (EAGLE design)
At the start: 72.8 x 77.5 mm, 64 parts, among them IC1 74HC125D, J1.1 MY_JUMPER, J1.2 MY_JUMPER, J2.2 10k, J6 MY_JUMPER, J7 MY_JUMPER

Commit message: Update PCB files
Parts:
- added GND_MAV: (no value), wirepad:SMD1,27-2,54
- moved CS 5.08 mm to (13.3, 47.6)
- moved B 4.45 mm to (13.3, 59.1)
- moved C 4.45 mm to (13.3, 53.3)
- moved R7 4.27 mm to (18.4, 40.6), turned to 270 degrees
- moved R 3.18 mm to (13.3, 55.2), turned to 90 degrees
- moved R6 2.14 mm to (21.0, 40.6), turned to 270 degrees
- moved AUDIO 1.27 mm to (13.3, 43.8)
- moved CTRL.DATA 1.27 mm to (13.3, 36.8)
- moved CTRL.LATCH 1.27 mm to (13.3, 38.7)
- moved PPUV 1.27 mm to (13.3, 45.7)
- moved 1 1.27 mm to (13.3, 26.7)
- moved 2 1.27 mm to (13.3, 28.6)
- moved 3 1.27 mm to (13.3, 30.5)
- moved CTRL.CLK 1.27 mm to (13.3, 40.6)
- moved RESET_OUT 1.27 mm to (13.3, 33.7)
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Connections:
- net GND: now also GND_MAV.1
Routing:
- net GND: track 28.6 -> 131.6 mm, vias 85 -> 88
- net AC2: track 26.9 -> 46.1 mm
- net AC1B: track 14.2 -> 33.4 mm
- net VCC: track 154.6 -> 167.2 mm
- net AC1A: track 18.5 -> 30.1 mm
- net DC2: track 39.8 -> 45.1 mm
- net N$1: track 23.4 -> 27.8 mm
- net N$5: track 98.1 -> 93.9 mm, vias 1 -> 2
- net N$11: track 14.1 -> 17.9 mm
- net N$20: track 9.26 -> 5.48 mm
- net N$28: track 13.3 -> 17.0 mm
- net N$35: track 20.5 -> 24.1 mm
- net N$3: track 29.1 -> 25.7 mm
- net N$6: track 20.8 -> 24.1 mm
- net N$34: track 27.6 -> 30.9 mm
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- added copper zone on layer 16, net N$30
Other:
- board text added: "CS"
- board text added: "Cr"
- board text added: "R6|R7"
- board text added: "Version: 20160420US"
- board text removed: "#CS"
- board text removed: "R6"
- board text removed: "R7"
- board text removed: "Version: 20151228US"
